Commit message: up

File: ros2_bipedal_ws/src/bipedal_robot_description/description/include.xacro (robot description, xacro)
@@ -11,4 +11,7 @@
     <material name="blue">
         <color rgba="0.2 0.2 1 1"/>
+    </material>
+	    <material name="red">
+        <color rgba="1 0.2 0.2 1"/>
     </material>
     <!-- Specify some standard inertial calculations https://en.wikipedia.org/wiki/List_of_moments_of_inertia -->
